File: TFT_adapter_BB.brd (EAGLE design)
At the start: 26.6 x 20 mm, 3 parts

Commit message: Finished the coprocessor
Parts:
- added U$1: CBT3244AD, custom:S020-75MM
Connections:
- new net VCC: U$1.P$20
- net GND: now also U$1.P$10
Other:
- board size 26.6 x 20 mm -> 43.2 x 20 mm
Changed lines of the file:
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@@
 <board>
 <plain>
-<wire x1="0" y1="0" x2="26.65" y2="0" width="0" layer="20"/>
-<wire x1="26.65" y1="0" x2="26.65" y2="19.99" width="0" layer="20"/>
-<wire x1="26.65" y1="19.99" x2="0" y2="19.99" width="0" layer="20"/>
+<wire x1="0" y1="0" x2="43.16" y2="0" width="0" layer="20"/>
+<wire x1="43.16" y1="0" x2="43.16" y2="19.99" width="0" layer="20"/>
+<wire x1="43.16" y1="19.99" x2="0" y2="19.99" width="0" layer="20"/>
 <wire x1="0" y1="19.99" x2="0" y2="0" width="0" layer="20"/>
 </plain>
@@
 <element name="J2" library="SparkFun-Connectors" package="1X09_NO_SILK" value="" x="22.86" y="17.78" rot="R180"/>
 <element name="TFT1" library="custom" package="TFT-CONN-18" value="TFT-18-1.0MM" x="13.97" y="8.89"/>
+<element name="U$1" library="custom" package="S020-75MM" value="CBT3244AD" x="34.29" y="15.24"/>
 </elements>
 <signals>
@@
 <wire x1="18.9738" y1="2.7432" x2="19.05" y2="2.54" width="0.254" layer="1"/>
 <wire x1="10.9728" y1="10.7442" x2="10.97" y2="10.89" width="0.254" layer="1"/>
+<contactref element="U$1" pad="P$10"/>
+<wire x1="19.05" y1="2.54" x2="30.48" y2="3.81" width="0" layer="19" extent="1-1"/>
 </signal>
 <signal name="N$2">
@@
 <wire x1="10.287" y1="17.6022" x2="10.16" y2="17.78" width="0.254" layer="1"/>
 </signal>
+<signal name="VCC">
+<contactref element="U$1" pad="P$20"/>
+</signal>
 </signals>
