File: coprocessor.sch (EAGLE design)
At the start: 49 parts, among them IC1 MEGA32U2, J1 AVR_SPI_PRG_6NS, U1 TPS61090RSAR, U3 V_REG_LDOSMD2, U4 AZV321, U5 MCP48, U6 16MHZ, U7 CBT3244AD

Commit message: added new gerbers and ordered the board
Parts:
- added U$2: LOGO2INCH_SVG, custom:LOGO2INCH_SVG
Changed lines of the file:
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@@
 <part name="SUPPLY24" library="SparkFun-Aesthetics" deviceset="V_USB" device=""/>
 <part name="SUPPLY10" library="SparkFun-Aesthetics" deviceset="VCC" device=""/>
+<part name="U$2" library="custom" deviceset="LOGO" device="2INCH_SVG"/>
 </parts>
 <sheets>
@@
 <instance part="SUPPLY25" gate="G$1" x="68.58" y="5.08"/>
 <instance part="GND29" gate="1" x="101.6" y="0"/>
+<instance part="U$2" gate="G$1" x="129.54" y="-17.78"/>
 </instances>
 <busses>
